File: mediaKeeb_V2/mediaKeeb_V2.kicad_pcb (KiCad board)
At the start: 2 copper layers, 75 x 50 mm, 18 parts, among them J1 Conn_01x05_Pin, SW1 SW_Push_45deg, SW2 SW_Push_45deg, SW3 SW_Push_45deg, SW4 SW_Push_45deg, SW5 SW_Push_45deg, SW6 SW_Push_45deg

Commit message: asd
Parts:
- removed J1: Conn_01x05_Pin, Connector_PinHeader_2.54mm:PinHeader_1x05_P2.54mm_Vertical
- added H1: MountingHole, MountingHole:MountingHole_3.2mm_M3, F.Cu at (215.1, 37.1)
- added H2: MountingHole, MountingHole:MountingHole_3.2mm_M3, F.Cu at (215.1, 45.1)
- added H3: MountingHole, MountingHole:MountingHole_3.2mm_M3, F.Cu at (215.1, 53.0)
- added H4: MountingHole, MountingHole:MountingHole_3.2mm_M3, F.Cu at (215.1, 61.0)
- added U1: ATmega32U4-A, Package_QFP:TQFP-44_10x10mm_P0.8mm, F.Cu at (261.8, 83.3)
- moved D4 3.81 mm to (138.4, 114.2)
- moved D3 3.76 mm to (176.4, 95.2)
- moved D2 3.76 mm to (157.4, 95.2)
- moved D5 3.76 mm to (157.4, 114.2)
- moved D6 3.74 mm to (176.4, 114.2)
- moved SW1 3.73 mm to (130.3, 88.1)
- moved SW2 3.73 mm to (149.3, 88.1)
- moved SW3 3.73 mm to (168.3, 88.1)
- moved SW4 3.73 mm to (130.3, 107.1)
- moved SW5 3.73 mm to (149.3, 107.1)
- moved SW6 3.73 mm to (168.3, 107.1)
- moved D1 3.72 mm to (138.3, 95.2)
Connections:
- D1 pad 1: (no net) -> Row_1
- D1 pad 2: (no net) -> Net-(D1-A)
- D2 pad 1: (no net) -> Row_1
- D2 pad 2: (no net) -> Net-(D2-A)
- D3 pad 1: (no net) -> Row_1
- D3 pad 2: (no net) -> Net-(D3-A)
- D4 pad 1: (no net) -> Row_2
- D4 pad 2: (no net) -> Net-(D4-A)
- D5 pad 1: (no net) -> Row_2
- D5 pad 2: (no net) -> Net-(D5-A)
- D6 pad 1: (no net) -> Row_2
- D6 pad 2: (no net) -> Net-(D6-A)
- SW1 pad 1: (no net) -> Column_1
- SW1 pad 2: (no net) -> Net-(D1-A)
- SW2 pad 1: (no net) -> Column_2
- SW2 pad 2: (no net) -> Net-(D2-A)
- SW3 pad 1: (no net) -> Column_3
- SW3 pad 2: (no net) -> Net-(D3-A)
- SW4 pad 1: (no net) -> Column_1
- SW4 pad 2: (no net) -> Net-(D4-A)
- SW5 pad 1: (no net) -> Column_2
- SW5 pad 2: (no net) -> Net-(D5-A)
- SW6 pad 1: (no net) -> Column_3
- SW6 pad 2: (no net) -> Net-(D6-A)
Routing:
- net (no net): track 388.3 -> 0.00 mm
Other:
- board text removed: "Col_1"
- board text removed: "Col_2"
- board text removed: "Col_3"
- board text removed: "Row_1"
- board text removed: "Row_2"
